File: Temperature Controlled FAN.kicad_sch (KiCad schematic)
At the start: 8 parts, among them J1 Input Voltage, J2 Fan Terminal, Q1 MJE13005G, U1 LM741

Commit message: Temperature controlled Fan is restored
Other:
- company: (none) -> by Muxtar_Safarov
- title: (none) -> Temperature controlled Fan 
Changed lines of the file:
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@@
 (kicad_sch (version 20230121) (generator eeschema)
   (paper "A4")
+  (title_block
+    (title "Temperature controlled Fan ")
+    (date "16.10.2022")
+    (rev "1.0")
+    (company "by Muxtar_Safarov")
+  )
   (junction (at 82.55 59.69) (diameter 0) (color 0 0 0 0)
   )
